File: pcb/out/ESP32_DevBoard/ESP32_DevBoard.kicad_pcb (KiCad board)
At the start: 2 copper layers, 50.6 x 53.2 mm, 15 parts, among them J1 USB_Micro-B, J2 UART, J3 GPIO, SW1 EN, SW2 BOOT, U1 ESP32-WROOM-32, U2 AMS1117-3.3

Commit message: HomeController PRO: sterownik domowy 32 wej / 16 wyj (2 plyty, 24V)
Nowe czesci: ESP32-C3 (modul kastelowany), TJA1051 (CAN), MOV (warystor),
MOSFET mocy DPAK (TO-252). Nowe bloki: wyjscie przekaznikowe 230V, wyjscie
MOSFET DC, bank wejsc RJ45 (TVS/wejscie), RS485, CAN, ESP32-C3, zlacze TFT.

Plyta DOLNA: 24V (bezpiecznik+dioda+MOV+buck5V+LDO3V3), ekspander wyjsc,
8x przekaznik 230V + 8x MOSFET DC, kazde wlasny zacisk; przekazniki we wnetrzu.
Plyta GORNA (wezsza): ESP32-C3 + 2x ekspander (32 wejscia), 8x RJ45, RS485+CAN,
TFT dotykowy. Otwory + B2B wspolne 1:1.

Layout: I/O na krawedzi dla OBU plyt (omija otwory narozne), zaciski 230V na
dolnej krawedzi, przekazniki we wnetrzu. Heurystyka zasilania rozpoznaje V24/Vxx;
regula diod tylko dla zlacz polowych (RJ45/zaciski). Niezawodnosc: TVS na kazdym
I/O, MOV, diody gasnace, pull-down bramek, grube sciezki 230V.

Oba PCB 0/0/0, zwalidowane kiutils (140 i 77 footprintow). Testy 12/12.

Co-Authored-By: Claude Opus 4.8 (1M context) <noreply@anthropic.com>
Claude-Session: https://claude.ai/code/session_01LNGxtK2Jv1rJLBLPTwFQ9C
Other:
- board text added: "ESP32_DevBoard"
Changed lines of the file:
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@@
     (layer "Edge.Cuts")
   )
+  (gr_text
+    "ESP32_DevBoard"
+    (at 2 51.7 0)
+    (layer "F.SilkS")
+    (effects
+      (font
+        (size 1.5 1.5)
+        (thickness 0.25)
+      )
+      (justify left)
+    )
+  )
 )
