File: pcb/out/HomeCtrl_Top/HomeCtrl_Top.kicad_sch (KiCad schematic)
At the start: 15 parts, among them J1 B2B, J2 RJ45-A, J3 RJ45-B, J4 RJ45-C, J5 RJ45-D, J6 GPIO, U1 MCP23017, U2 DS18B20

Commit message: HomeController PRO: sterownik domowy 32 wej / 16 wyj (2 plyty, 24V)
Nowe czesci: ESP32-C3 (modul kastelowany), TJA1051 (CAN), MOV (warystor),
MOSFET mocy DPAK (TO-252). Nowe bloki: wyjscie przekaznikowe 230V, wyjscie
MOSFET DC, bank wejsc RJ45 (TVS/wejscie), RS485, CAN, ESP32-C3, zlacze TFT.

Plyta DOLNA: 24V (bezpiecznik+dioda+MOV+buck5V+LDO3V3), ekspander wyjsc,
8x przekaznik 230V + 8x MOSFET DC, kazde wlasny zacisk; przekazniki we wnetrzu.
Plyta GORNA (wezsza): ESP32-C3 + 2x ekspander (32 wejscia), 8x RJ45, RS485+CAN,
TFT dotykowy. Otwory + B2B wspolne 1:1.

Layout: I/O na krawedzi dla OBU plyt (omija otwory narozne), zaciski 230V na
dolnej krawedzi, przekazniki we wnetrzu. Heurystyka zasilania rozpoznaje V24/Vxx;
regula diod tylko dla zlacz polowych (RJ45/zaciski). Niezawodnosc: TVS na kazdym
I/O, MOV, diody gasnace, pull-down bramek, grube sciezki 230V.

Oba PCB 0/0/0, zwalidowane kiutils (140 i 77 footprintow). Testy 12/12.

Co-Authored-By: Claude Opus 4.8 (1M context) <noreply@anthropic.com>
Claude-Session: https://claude.ai/code/session_01LNGxtK2Jv1rJLBLPTwFQ9C
Changed lines of the file:
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@@
         "HomeCtrl_Top"
         (path
-          "/00b6cf25-b3f6-494e-a21c-41606a1e66b7"
+          "/96bfc4fe-5b48-43aa-95aa-a66a7135746a"
           (reference "J1")
           (unit 1)
@@
         "HomeCtrl_Top"
         (path
-          "/00b6cf25-b3f6-494e-a21c-41606a1e66b7"
+          "/96bfc4fe-5b48-43aa-95aa-a66a7135746a"
           (reference "U1")
           (unit 1)
@@
         "HomeCtrl_Top"
         (path
-          "/00b6cf25-b3f6-494e-a21c-41606a1e66b7"
+          "/96bfc4fe-5b48-43aa-95aa-a66a7135746a"
           (reference "C1")
           (unit 1)
@@
         "HomeCtrl_Top"
         (path
-          "/00b6cf25-b3f6-494e-a21c-41606a1e66b7"
+          "/96bfc4fe-5b48-43aa-95aa-a66a7135746a"
           (reference "R1")
           (unit 1)
@@
         "HomeCtrl_Top"
         (path
-          "/00b6cf25-b3f6-494e-a21c-41606a1e66b7"
+          "/96bfc4fe-5b48-43aa-95aa-a66a7135746a"
           (reference "R2")
           (unit 1)
@@
         "HomeCtrl_Top"
         (path
-          "/00b6cf25-b3f6-494e-a21c-41606a1e66b7"
+          "/96bfc4fe-5b48-43aa-95aa-a66a7135746a"
           (reference "R3")
           (unit 1)
@@
         "HomeCtrl_Top"
         (path
-          "/00b6cf25-b3f6-494e-a21c-41606a1e66b7"
+          "/96bfc4fe-5b48-43aa-95aa-a66a7135746a"
           (reference "U2")
           (unit 1)
@@
         "HomeCtrl_Top"
         (path
-          "/00b6cf25-b3f6-494e-a21c-41606a1e66b7"
+          "/96bfc4fe-5b48-43aa-95aa-a66a7135746a"
           (reference "J2")
           (unit 1)
@@
         "HomeCtrl_Top"
         (path
-          "/00b6cf25-b3f6-494e-a21c-41606a1e66b7"
+          "/96bfc4fe-5b48-43aa-95aa-a66a7135746a"
           (reference "J3")
           (unit 1)
@@
         "HomeCtrl_Top"
         (path
-          "/00b6cf25-b3f6-494e-a21c-41606a1e66b7"
+          "/96bfc4fe-5b48-43aa-95aa-a66a7135746a"
           (reference "J4")
           (unit 1)
@@
         "HomeCtrl_Top"
         (path
-          "/00b6cf25-b3f6-494e-a21c-41606a1e66b7"
+          "/96bfc4fe-5b48-43aa-95aa-a66a7135746a"
           (reference "J5")
           (unit 1)
@@
         "HomeCtrl_Top"
         (path
-          "/00b6cf25-b3f6-494e-a21c-41606a1e66b7"
+          "/96bfc4fe-5b48-43aa-95aa-a66a7135746a"
           (reference "J6")
           (unit 1)
@@
         "HomeCtrl_Top"
         (path
-          "/00b6cf25-b3f6-494e-a21c-41606a1e66b7"
+          "/96bfc4fe-5b48-43aa-95aa-a66a7135746a"
           (reference "D1")
           (unit 1)
@@
         "HomeCtrl_Top"
         (path
-          "/00b6cf25-b3f6-494e-a21c-41606a1e66b7"
+          "/96bfc4fe-5b48-43aa-95aa-a66a7135746a"
           (reference "D2")
           (unit 1)
@@
         "HomeCtrl_Top"
         (path
-          "/00b6cf25-b3f6-494e-a21c-41606a1e66b7"
+          "/96bfc4fe-5b48-43aa-95aa-a66a7135746a"
           (reference "D3")
           (unit 1)
@@
         "HomeCtrl_Top"
         (path
-          "/00b6cf25-b3f6-494e-a21c-41606a1e66b7"
+          "/96bfc4fe-5b48-43aa-95aa-a66a7135746a"
           (reference "#FLG?")
           (unit 1)
@@
         "HomeCtrl_Top"
         (path
-          "/00b6cf25-b3f6-494e-a21c-41606a1e66b7"
+          "/96bfc4fe-5b48-43aa-95aa-a66a7135746a"
           (reference "#FLG?")
           (unit 1)
@@
     (fields_autoplaced)
     (effects
+      (font
+        (size 1.27 1.27)
+      )
+    )
+  )
+  (symbol
+    (lib_id "pcbforge:PWR_FLAG")
+    (at 250 49 0)
+    (unit 1)
+    (exclude_from_sim no)
+    (in_bom no)
+    (on_board yes)
+    (dnp no)
+    (property
+      "Reference"
+      "#FLG?"
+      (at 250 46 0)
+      (effects
+        (font
+          (size 1.27 1.27)
+        )
+        (hide yes)
+      )
+    )
+    (property
+      "Value"
+      "PWR_FLAG"
+      (at 250 52 0)
+      (effects
+        (font
+          (size 1.27 1.27)
+        )
+      )
+    )
+    (property
+      "Footprint"
+      ""
+      (at 250 49 0)
+      (effects
+        (font
+          (size 1.27 1.27)
+        )
+        (hide yes)
+      )
+    )
+    (property
+      "Datasheet"
+      ""
+      (at 250 49 0)
+      (effects
+        (font
+          (size 1.27 1.27)
+        )
+        (hide yes)
+      )
+    )
+    (pin
+      "1"
+    )
+    (instances
+      (project
+        "HomeCtrl_Top"
+        (path
+          "/96bfc4fe-5b48-43aa-95aa-a66a7135746a"
+          (reference "#FLG?")
+          (unit 1)
+        )
+      )
+    )
+  )
+  (global_label
+    "V5"
+    (shape bidirectional)
+    (at 250 49 0)
+    (fields_autoplaced)
+    (effects
