File: pcb/out/SmartHome230_Bottom/SmartHome230_Bottom.kicad_sch (KiCad schematic)
At the start: 56 parts, among them J1 12V IN, J2 UART, J3 RJ45-A, J4 RJ45-B, J5 RJ45-C, J6 RJ45-D, SW1 EN, SW2 BOOT, U1 MP1584, U2 AMS1117-3.3, U3 ESP32-WROOM-32, U4 MCP23017, U5 DS18B20

Commit message: Zasady rozmieszczania: I/O na krawedziach, strefa 230V, plyty gora/dol
Wdrozone zasady uzytkownika (pcbforge/layout.py + smart_home_230.py):
- I/O (zlacza) na gornej krawedzi; przekazniki + zaciski 230V w osobnej strefie
  na dolnej krawedzi (izolacja od logiki).
- otwory montazowe i zlacze board-to-board w IDENTYCZNYCH wspolrzednych na obu
  plytkach (wspolna Frame) - skladaja sie 1:1.
- gorna plytka WEZSZA o pasy I/O (Design.outline = srodek) - dostep srubokretem
  do zaciskow dolnej plytki.
- osobna dioda/TVS na kazde I/O (regula DIODE_PER_IO).
- 230V: design.mark_mains() -> klasa 'mains' w DSN (1.5mm sciezki, 2.5mm izolacja);
  regula MAINS_UNMARKED pilnuje oznaczenia kontaktow przekaznikow.
- pasywne od spodu (poprawne warstwy B.* + lustro padow w pcb_writer).
- opisy po polsku na silku (Component.label, Design.notes).

Nowe czesci: przekaznik SPDT (szerokie pady 230V), otwor montazowy M3, blok
relay_driver. Reguly swiadome zlacza B2B (sieci miedzyplytkowe nie flagowane).
9 zasad zapisane trwale w knowledge/kb.json. Flagowiec SmartHome230 (2 plyty):
ERC/DRC/reguly 0/0/0, zwalidowane kiutils. Testy 11/11.

Co-Authored-By: Claude Opus 4.8 (1M context) <noreply@anthropic.com>
Claude-Session: https://claude.ai/code/session_01LNGxtK2Jv1rJLBLPTwFQ9C
Parts:
- removed C14: 100nF, pcbforge:C_0805, symbol pcbforge:C
- removed D12, D13, D14, D15, D16, D17, D18, D19: ESD, pcbforge:D_SOD-323, symbol pcbforge:D_TVS
- removed J1: 12V IN, pcbforge:ScrewTerminal_1x02, symbol pcbforge:ScrewTerminal_1x02
- removed J2: UART, pcbforge:Header_1x06, symbol pcbforge:Header_1x06
- removed J5: RJ45-C, pcbforge:RJ45_8P8C, symbol pcbforge:RJ45_8P8C
- removed J6: RJ45-D, pcbforge:RJ45_8P8C, symbol pcbforge:RJ45_8P8C
- removed U4: MCP23017, pcbforge:SOIC-28, symbol pcbforge:MCP23017
- removed U5: DS18B20, pcbforge:TO-92, symbol pcbforge:DS18B20
- added D12, D13: 1N4148, pcbforge:D_SMA, symbol pcbforge:D
- added H1, H2, H3, H4: M3, pcbforge:MountingHole_M3, symbol pcbforge:MountingHole
- added J1: B2B, pcbforge:Header_2x10, symbol pcbforge:Header_2x10
- added J2: 12V, pcbforge:ScrewTerminal_1x02, symbol pcbforge:ScrewTerminal_1x02
- added J5: UART, pcbforge:Header_1x06, symbol pcbforge:Header_1x06
- added J6: 230V IN, pcbforge:ScrewTerminal_1x03, symbol pcbforge:ScrewTerminal_1x03
- added J7: Wyj.1, pcbforge:ScrewTerminal_1x03, symbol pcbforge:ScrewTerminal_1x03
- added J8: Wyj.2, pcbforge:ScrewTerminal_1x03, symbol pcbforge:ScrewTerminal_1x03
- added K1, K2: SRD-12V, pcbforge:Relay_SPDT_SRD, symbol pcbforge:Relay_SPDT
- added Q1, Q2: BC547, pcbforge:SOT-23-3, symbol pcbforge:Q_NPN
- added R9: 1k, pcbforge:R_0805, symbol pcbforge:R
- J3: value RJ45-A -> Przyciski A
- J4: value RJ45-B -> Przyciski B
- R5: value 4.7k -> 10k
- R8: value 10k -> 1k
Connections:
- net 3V3: now also J1.19 (P19), J1.3 (P3), J1.4 (P4), J5.2 (P2); no longer R8.1
- net BTN0: now also D3.1, J1.10 (P10); no longer D4.1
- net BTN1: now also D4.1, J1.11 (P11); no longer D5.1
- net BTN2: now also D5.1, J1.12 (P12); no longer D6.1
- net BTN3: now also D6.1, J1.13 (P13); no longer D7.1
- net BTN4: now also D7.1, J1.14 (P14); no longer D8.1
- net BTN5: now also D8.1, J1.15 (P15); no longer D9.1
- net BTN6: now also D9.1, J1.16 (P16); no longer D10.1
- net BTN7: now also D10.1, J1.17 (P17); no longer D11.1
- net EN: now also J5.3 (P3)
- net EXP_INT: now also J1.7 (P7)
- net EXP_RST: now also R5.2, J1.8 (P8); no longer R8.2
- net GND: now also J1.1 (P1), J1.18 (P18), J1.2 (P2), J1.20 (P20), J2.2, J5.1 (P1), Q1.3 (E), Q2.3 (E)
- net IO0: now also J5.4 (P4)
- net OW: now also D11.1, U3.13 (IO14), J1.9 (P9); no longer D3.1, R7.2, U3.26 (IO4)
- net RXD0: now also J5.6 (P6)
- net SCL: now also R7.2, J1.6 (P6); no longer R6.2
- net SDA: now also R6.2, J1.5 (P5); no longer R5.2
- net TXD0: now also J5.5 (P5)
- net VIN: now also J2.1
- net RELAY2: now reaches U3.29 (IO5)
- net RELAY2: now also R9.1
- net VIN_P renamed V12
- net V12: now also D12.2, D13.2, K1.1 (COIL+), K2.1 (COIL+)
- net _FUSED_VIN_P renamed _FUSED_V12
- new net L: J6.1, K1.4 (COM), K2.4 (COM)
- new net LAMP1: J7.1, K1.3 (NO)
- new net LAMP2: J8.1, K2.3 (NO)
- new net N: J6.2, J7.2, J8.2
- new net PE: J6.3, J7.3, J8.3
- new net RELAY1: R8.1, U3.26 (IO4)
- new net _B_LAMP1: Q1.1 (B), R8.2
- new net _B_LAMP2: Q2.1 (B), R9.2
- new net _COIL_LAMP1: D12.1, K1.2 (COIL-), Q1.2 (C)
- new net _COIL_LAMP2: D13.1, K2.2 (COIL-), Q2.2 (C)
