File: pcb/out/HomeCtrlPro_Bottom/HomeCtrlPro_Bottom.kicad_sch (KiCad schematic)
At the start: 140 parts, among them J1 B2B, J10 OUT6, J11 OUT7, J12 OUTDC8, J13 OUTDC9, J14 OUTDC10, J15 OUTDC11, J16 OUTDC12, J17 OUTDC13, J18 OUTDC14, J19 OUTDC15, J2 24V, J3 230V, J4 OUT0, J5 OUT1, J6 OUT2, J7 OUT3, J8 OUT4, J9 OUT5, K1 SRD-24V, K2 SRD-24V, K3 SRD-24V, K4 SRD-24V, K5 SRD-24V, K6 SRD-24V, K7 SRD-24V, K8 SRD-24V, Q1 BC547, Q10 IRLZ44N, Q11 IRLZ44N, Q12 IRLZ44N, Q13 IRLZ44N, Q14 IRLZ44N, Q15 IRLZ44N, Q16 IRLZ44N, Q2 BC547, Q3 BC547, Q4 BC547, Q5 BC547, Q6 BC547, Q7 BC547, Q8 BC547, Q9 IRLZ44N, U1 MP1584, U2 AMS1117-3.3, U3 MCP23017

Commit message: Wiecej RJ45 (8 podwojnych=64 wej), zabezpieczenia, zlacza na obu krawedziach
- Wejscia: 8 podwojnych RJ45 = 16 portow = 64 wejscia (4 ekspandery MCP23017).
- Zabezpieczenia: PTC na kazde z 16 wyjsc, MOV na wyjsciach 230V, snubber RC na
  stykach przekaznikow, dlawik wspolny (CMC) + TVS na RS485/CAN, TVS na wyjsciach DC.
  Nowe czesci: PTC (polyfuse), CMC (common-mode choke).
- Layout: zlacza rozlozone na GORNA i DOLNA krawedz (_split_balanced) -> wezsza
  plytka; gestsze upakowanie, mniejszy luz wysokosci. auto_frame liczy szerokosc
  z rozlozenia na 2 krawedzie. HomeCtrlPro: 237 -> 155 mm szerokosci.

Oba PCB 0/0/0, testy 12/12, kiutils OK.

Co-Authored-By: Claude Opus 4.8 (1M context) <noreply@anthropic.com>
Claude-Session: https://claude.ai/code/session_01LNGxtK2Jv1rJLBLPTwFQ9C
Parts:
- removed D12, D14, D16, D18: SS34, pcbforge:D_SMA, symbol pcbforge:D_Schottky
- added C12, C13, C14, C15, C16, C17, C18, C19: 100nF, pcbforge:C_0805, symbol pcbforge:C
- added D12, D14, D16, D18, D20, D22, D24, D26: TVS, pcbforge:D_SOD-323, symbol pcbforge:D_TVS
- added D19, D21, D23, D25: SS34, pcbforge:D_SMA, symbol pcbforge:D_Schottky
- added F10, F11, F12, F13, F14, F15, F16, F17: 2A, pcbforge:PTC_1812, symbol pcbforge:PTC
- added F2, F3, F4, F5, F6, F7, F8, F9: 0.5A, pcbforge:PTC_1812, symbol pcbforge:PTC
- added R43, R46, R49: 100k, pcbforge:R_0805, symbol pcbforge:R
- added R44, R47, R50: 1k, pcbforge:R_0805, symbol pcbforge:R
- added R45, R48: 100, pcbforge:R_0805, symbol pcbforge:R
- added RV2, RV3, RV4, RV5, RV6, RV7, RV8, RV9: S14K275, pcbforge:MOV_Disc, symbol pcbforge:MOV
- R11, R14, R17, R27, R30, R33, R36, R39, R42, R5, R8: value 1k -> 100
- R19, R22, R25: value 100 -> 1k
- R20, R23, R26: value 100k -> 100
- R28, R31, R34, R37, R40: value 100 -> 100k
- R29, R32, R35, R38, R41: value 100k -> 1k
Connections:
- net 3V3: now also U3.17 (A2); no longer U3.16 (A1)
- net GND: now also R28.2, R31.2, R34.2, R37.2, R40.2, U3.16 (A1), D12.2, D14.2, D16.2, D18.2, D20.2, D22.2, D24.2, D26.2, R43.2, R46.2, R49.2; no longer R20.2, R23.2, R26.2, R29.2, R32.2, R35.2, R38.2, R41.2, U3.17 (A2)
- net L: now also R11.1, R14.1, R17.1, R20.1, R23.1, R26.1, R5.1, R8.1
- net LAMP0: now also F2.2, RV2.1; no longer K1.3 (NO)
- net LAMP1: now also F3.2, RV3.1; no longer K2.3 (NO)
- net LAMP2: now also F4.2, RV4.1; no longer K3.3 (NO)
- net LAMP3: now also F5.2, RV5.1; no longer K4.3 (NO)
- net LAMP4: now also F6.2, RV6.1; no longer K5.3 (NO)
- net LAMP5: now also F7.2, RV7.1; no longer K6.3 (NO)
- net LAMP6: now also F8.2, RV8.1; no longer K7.3 (NO)
- net LAMP7: now also F9.2, RV9.1; no longer K8.3 (NO)
- net N: now also RV2.2, RV3.2, RV4.2, RV5.2, RV6.2, RV7.2, RV8.2, RV9.2
- net OUT1: now also R7.1; no longer R5.1
- net OUT10: now also R33.1, R35.1; no longer D13.1, J14.2, Q11.2 (D), R25.1, R27.1
- net OUT11: now also R36.1, R38.1; no longer J15.2, Q12.2 (D), R28.1, R30.1
- net OUT12: now also R39.1, R41.1; no longer D15.1, J16.2, Q13.2 (D), R31.1, R33.1
- net OUT13: now also R42.1, R44.1; no longer J17.2, Q14.2 (D), R34.1, R36.1
- net OUT14: now also R45.1, R47.1; no longer D17.1, J18.2, Q15.2 (D), R37.1, R39.1
- net OUT15: now also R48.1, R50.1; no longer J19.2, Q16.2 (D), R40.1, R42.1
- net OUT2: now also R10.1, R9.1; no longer R7.1, R8.1
- net OUT3: now also R12.1, R13.1; no longer R10.1, R9.1
- net OUT4: now also R15.1, R16.1; no longer R11.1, R12.1
- net OUT5: now also R18.1, R19.1; no longer R13.1, R14.1
- net OUT6: now also R21.1, R22.1; no longer R15.1, R16.1
- net OUT7: now also R24.1, R25.1; no longer R17.1, R18.1
- net OUT8: now also R27.1, R29.1; no longer D11.1, J12.2, Q9.2 (D), R19.1, R21.1
- net OUT9: now also R30.1, R32.1; no longer J13.2, Q10.2 (D), R22.1, R24.1
- net V24P: now also D19.2, D21.2, D23.2, D25.2
- net _G10: now also R33.2, R34.1; no longer R25.2, R26.1
- net _G11: now also R36.2, R37.1; no longer R28.2, R29.1
- net _G12: now also R39.2, R40.1; no longer R31.2, R32.1
- net _G13: now also R42.2, R43.1; no longer R34.2, R35.1
- net _G14: now also R45.2, R46.1; no longer R37.2, R38.1
- net _G15: now also R48.2, R49.1; no longer R40.2, R41.1
- net _G8: now also R27.2, R28.1; no longer R19.2, R20.1
- net _G9: now also R30.2, R31.1; no longer R22.2, R23.1
- net _ML10: now also R35.2; no longer R27.2
- net _ML11: now also R38.2; no longer R30.2
- net _ML12: now also R41.2; no longer R33.2
- net _ML13: now also R44.2; no longer R36.2
- net _ML14: now also R47.2; no longer R39.2
- net _ML15: now also R50.2; no longer R42.2
- net _ML8: now also R29.2; no longer R21.2
- net _ML9: now also R32.2; no longer R24.2
- net _RB1: now also R6.2; no longer R5.2
- net _RB2: now also R9.2; no longer R7.2
- net _RB3: now also R12.2; no longer R9.2
- net _RB4: now also R15.2; no longer R11.2
- net _RB5: now also R18.2; no longer R13.2
- net _RB6: now also R21.2; no longer R15.2
- net _RB7: now also R24.2; no longer R17.2
- net _RL1: now also R7.2; no longer R6.2
- net _RL2: now also R10.2; no longer R8.2
- net _RL3: now also R13.2; no longer R10.2
- net _RL4: now also R16.2; no longer R12.2
- net _RL5: now also R19.2; no longer R14.2
- net _RL6: now also R22.2; no longer R16.2
- net _RL7: now also R25.2; no longer R18.2
- new net OUTDC10: D16.1, F12.2, J14.2
- new net OUTDC11: D18.1, F13.2, J15.2
- new net OUTDC12: D20.1, F14.2, J16.2
- new net OUTDC13: D22.1, F15.2, J17.2
- new net OUTDC14: D24.1, F16.2, J18.2
- new net OUTDC15: D26.1, F17.2, J19.2
- new net OUTDC8: D12.1, F10.2, J12.2
- new net OUTDC9: D14.1, F11.2, J13.2
- new net _DRN10: D15.1, F12.1, Q11.2 (D)
- new net _DRN11: D17.1, F13.1, Q12.2 (D)
- new net _DRN12: D19.1, F14.1, Q13.2 (D)
- new net _DRN13: D21.1, F15.1, Q14.2 (D)
- new net _DRN14: D23.1, F16.1, Q15.2 (D)
- new net _DRN15: D25.1, F17.1, Q16.2 (D)
- new net _DRN8: D11.1, F10.1, Q9.2 (D)
- new net _DRN9: D13.1, F11.1, Q10.2 (D)
- new net _NO0: C12.2, F2.1, K1.3 (NO)
- new net _NO1: C13.2, F3.1, K2.3 (NO)
- new net _NO2: C14.2, F4.1, K3.3 (NO)
- new net _NO3: C15.2, F5.1, K4.3 (NO)
- new net _NO4: C16.2, F6.1, K5.3 (NO)
- new net _NO5: C17.2, F7.1, K6.3 (NO)
- new net _NO6: C18.2, F8.1, K7.3 (NO)
- new net _NO7: C19.2, F9.1, K8.3 (NO)
- new net _SN0: C12.1, R5.2
- new net _SN1: C13.1, R8.2
- new net _SN2: C14.1, R11.2
- new net _SN3: C15.1, R14.2
- new net _SN4: C16.1, R17.2
- new net _SN5: C17.1, R20.2
- new net _SN6: C18.1, R23.2
- new net _SN7: C19.1, R26.2
