File: pcb/out/HomeCtrlPro_Top/HomeCtrlPro_Top.kicad_sch (KiCad schematic)
At the start: 77 parts, among them J1 B2B, J10 RS485, J11 CAN, J12 TFT, J2 Wejscia 0-3, J3 Wejscia 4-7, J4 Wejscia 8-11, J5 Wejscia 12-15, J6 Wejscia 16-19, J7 Wejscia 20-23, J8 Wejscia 24-27, J9 Wejscia 28-31, SW1 RST, SW2 BOOT, U1 ESP32-C3-MINI-1, U2 MCP23017, U3 MCP23017, U4 MAX485, U5 TJA1051

Commit message: ESP32-S3 + przyciski TFT; kompaktowy layout (szerokosc z liczby zlacz, 2 rzedy)
- Przejscie ESP32-C3 -> ESP32-S3 (duzo GPIO): niezalezne RS485/CAN, dotyk z IRQ,
  4 przyciski nawigacji TFT (GORA/DOL/OK/WSTECZ). Nowa czesc ESP32-S3-WROOM-1.
- Layout: I/O wzdluz krawedzi w 2 rzedach (podwojne w pionie), szerokosc plytki
  wynika z LICZBY zlacz (zmienne szerokosci kolumn) - wejscia na gornej krawedzi,
  wyjscia (zaciski) na dolnej. auto_frame() dobiera ciasna wspolna ramke.
- Przekazniki pakowane w strefe 230V (kilka rzedow) omijajaca otwory.
- HomeCtrlPro: 280x185 -> 168x192 mm, mniej pustego miejsca. Oba 0/0/0.

Testy 12/12, zwalidowane kiutils. Bloki: esp32s3, button.

Co-Authored-By: Claude Opus 4.8 (1M context) <noreply@anthropic.com>
Claude-Session: https://claude.ai/code/session_01LNGxtK2Jv1rJLBLPTwFQ9C
Parts:
- removed U1: ESP32-C3-MINI-1, pcbforge:ESP32-C3-MINI-1, symbol pcbforge:ESP32-C3-MINI-1
- added C8: 100nF, pcbforge:C_0805, symbol pcbforge:C
- added R11, R14: 120, pcbforge:R_0805, symbol pcbforge:R
- added R12, R13: 560, pcbforge:R_0805, symbol pcbforge:R
- added SW3: GORA, pcbforge:SW_Push_6mm, symbol pcbforge:SW_Push
- added SW4: DOL, pcbforge:SW_Push_6mm, symbol pcbforge:SW_Push
- added SW5: OK, pcbforge:SW_Push_6mm, symbol pcbforge:SW_Push
- added SW6: WSTECZ, pcbforge:SW_Push_6mm, symbol pcbforge:SW_Push
- added U1: ESP32-S3-WROOM-1, pcbforge:ESP32-S3-WROOM-1, symbol pcbforge:ESP32-S3-WROOM-1
- J2: value Wejscia 0-3 -> We 0-3
- J3: value Wejscia 4-7 -> We 4-7
- J4: value Wejscia 8-11 -> We 8-11
- J5: value Wejscia 12-15 -> We 12-15
- J6: value Wejscia 16-19 -> We 16-19
- J7: value Wejscia 20-23 -> We 20-23
- J8: value Wejscia 24-27 -> We 24-27
- J9: value Wejscia 28-31 -> We 28-31
- R10, R7: value 120 -> 10k
- R8, R9: value 560 -> 10k
Connections:
- net 3V3: now also C3.1, R10.1, R7.1, R9.1, C8.1, R12.1, U1.2 (3V3); no longer C4.1, J12.11 (P11), J12.4 (P4)
- net CAN_H: now also R14.1; no longer R10.1
- net CAN_L: now also R14.2; no longer R10.2
- net CAN_TXD: now also U1.8 (IO4)
- net EN: now also C4.1, U1.3 (EN); no longer C3.1
- net GND: now also C8.2, R13.2, SW3.3 (B), SW3.4 (B), SW4.3 (B), SW4.4 (B), SW5.3 (B), SW5.4 (B), SW6.3 (B), SW6.4 (B), U1.1 (GND), U1.40 (GND); no longer R9.2
- net RS485_A: now also R11.1, R12.2; no longer R7.1, R8.2
- net RS485_B: now also R11.2, R13.1; no longer R7.2, R9.1
- net RS485_DE: now also U1.36 (IO45)
- net RS485_RXD: now also U1.35 (IO44)
- net RS485_TXD: now also U1.34 (IO43)
- net SCL: now also U1.13 (IO9)
- net SDA: now also U1.12 (IO8)
- net SPI_MISO: now also U1.17 (IO13)
- net SPI_MOSI: now also U1.15 (IO11)
- net SPI_SCK: now also U1.16 (IO12)
- net TFT_CS: now also U1.14 (IO10)
- net TFT_DC: now also U1.18 (IO14)
- net TOUCH_CS: now also U1.38 (IO47)
- net EXP_INT: now reaches U2.20 (INTA)
- net EXP_INT: now also U3.20 (INTA), U1.21 (IO17)
- net IO9 renamed IO0
- net IO0: now also U1.4 (IO0); no longer U5.4 (RXD)
- new net BTN_BACK: R10.2, SW6.1 (A), SW6.2 (A), U1.20 (IO16)
- new net BTN_DOWN: R8.2, SW4.1 (A), SW4.2 (A), U1.11 (IO7)
- new net BTN_OK: R9.2, SW5.1 (A), SW5.2 (A), U1.19 (IO15)
- new net BTN_UP: R7.2, SW3.1 (A), SW3.2 (A), U1.10 (IO6)
- new net CAN_RXD: U1.9 (IO5), U5.4 (RXD)
- new net TFT_RST: J12.4 (P4), U1.25 (IO21)
- new net TOUCH_IRQ: J12.11 (P11), U1.39 (IO48)

Commit message: Wejscia w jednym rzedzie PRZY krawedzi + gniazda RJ45 podwojne (2 porty w pionie)
Poprawka po blednej interpretacji: I/O ustawiane w JEDNYM rzedzie zlicowanym do
krawedzi (koniec ze stosowaniem zlacz w 2 rzedach do wnetrza). Szerokosc plytki
= suma szerokosci zlacz w rzedzie. Nowa czesc RJ45_Dual (2 porty RJ45 w jednej
obudowie, jeden nad drugim) + blok input_bank_dual (8 wejsc/gniazdo, TVS/wejscie).
HomeCtrlPro: 4 podwojne RJ45 = 32 wejscia. Oba PCB 0/0/0, testy 12/12, kiutils OK.

Co-Authored-By: Claude Opus 4.8 (1M context) <noreply@anthropic.com>
Claude-Session: https://claude.ai/code/session_01LNGxtK2Jv1rJLBLPTwFQ9C
Parts:
- removed J10: RS485, pcbforge:RJ45_8P8C, symbol pcbforge:RJ45_8P8C
- removed J11: CAN, pcbforge:RJ45_8P8C, symbol pcbforge:RJ45_8P8C
- removed J12: TFT, pcbforge:Header_1x14, symbol pcbforge:Header_1x14
- removed J2: We 0-3, pcbforge:RJ45_8P8C, symbol pcbforge:RJ45_8P8C
- removed J3: We 4-7, pcbforge:RJ45_8P8C, symbol pcbforge:RJ45_8P8C
- removed J4: We 8-11, pcbforge:RJ45_8P8C, symbol pcbforge:RJ45_8P8C
- removed J5: We 12-15, pcbforge:RJ45_8P8C, symbol pcbforge:RJ45_8P8C
- removed J8: We 24-27, pcbforge:RJ45_8P8C, symbol pcbforge:RJ45_8P8C
- removed J9: We 28-31, pcbforge:RJ45_8P8C, symbol pcbforge:RJ45_8P8C
- added J2: We 0-7, pcbforge:RJ45_Dual, symbol pcbforge:RJ45_Dual
- added J3: We 8-15, pcbforge:RJ45_Dual, symbol pcbforge:RJ45_Dual
- added J4: We 16-23, pcbforge:RJ45_Dual, symbol pcbforge:RJ45_Dual
- added J5: We 24-31, pcbforge:RJ45_Dual, symbol pcbforge:RJ45_Dual
- added J8: TFT, pcbforge:Header_1x14, symbol pcbforge:Header_1x14
- J6: value We 16-19 -> RS485
- J7: value We 20-23 -> CAN
Connections:
- net 3V3: now also J6.7 (P7), J6.8 (P8), J7.7 (P7), J7.8 (P8), J2.1 (A1), J2.9 (B1), J3.1 (A1), J3.9 (B1), J4.1 (A1), J4.9 (B1), J5.1 (A1), J5.9 (B1), J8.14 (P14), J8.2 (P2), J8.8 (P8); no longer J6.1 (P1), J7.1 (P1)
- net CAN_H: now also J7.1 (P1)
- net CAN_L: now also J7.2 (P2)
- net GND: now also J6.3 (P3), J6.4 (P4), J6.5 (P5), J7.3 (P3), J7.4 (P4), J7.5 (P5), J2.14 (B6), J2.15 (B7), J2.16 (B8), J2.6 (A6), J2.7 (A7), J2.8 (A8), J2.S (SHIELD), J3.14 (B6), J3.15 (B7), J3.16 (B8), J3.6 (A6), J3.7 (A7), J3.8 (A8), J3.S (SHIELD), J4.14 (B6), J4.15 (B7), J4.16 (B8), J4.6 (A6), J4.7 (A7), J4.8 (A8), J4.S (SHIELD), J5.14 (B6), J5.15 (B7), J5.16 (B8), J5.6 (A6), J5.7 (A7), J5.8 (A8), J5.S (SHIELD), J8.1 (P1), J8.13 (P13); no longer J6.7 (P7), J6.8 (P8), J7.7 (P7), J7.8 (P8)
- net IN0: now also J2.2 (A2)
- net IN1: now also J2.3 (A3)
- net IN10: now also J3.4 (A4)
- net IN11: now also J3.5 (A5)
- net IN12: now also J3.10 (B2)
- net IN13: now also J3.11 (B3)
- net IN14: now also J3.12 (B4)
- net IN15: now also J3.13 (B5)
- net IN16: now also J4.2 (A2); no longer J6.2 (P2)
- net IN17: now also J4.3 (A3); no longer J6.3 (P3)
- net IN18: now also J4.4 (A4); no longer J6.4 (P4)
- net IN19: now also J4.5 (A5); no longer J6.5 (P5)
- net IN2: now also J2.4 (A4)
- net IN20: now also J4.10 (B2); no longer J7.2 (P2)
- net IN21: now also J4.11 (B3); no longer J7.3 (P3)
- net IN22: now also J4.12 (B4); no longer J7.4 (P4)
- net IN23: now also J4.13 (B5); no longer J7.5 (P5)
- net IN24: now also J5.2 (A2)
- net IN25: now also J5.3 (A3)
- net IN26: now also J5.4 (A4)
- net IN27: now also J5.5 (A5)
- net IN28: now also J5.10 (B2)
- net IN29: now also J5.11 (B3)
- net IN3: now also J2.5 (A5)
- net IN30: now also J5.12 (B4)
- net IN31: now also J5.13 (B5)
- net IN4: now also J2.10 (B2)
- net IN5: now also J2.11 (B3)
- net IN6: now also J2.12 (B4)
- net IN7: now also J2.13 (B5)
- net IN8: now also J3.2 (A2)
- net IN9: now also J3.3 (A3)
- net RS485_A: now also J6.1 (P1)
- net RS485_B: now also J6.2 (P2)
- net SPI_MISO: now also J8.12 (P12), J8.9 (P9)
- net SPI_MOSI: now also J8.6 (P6)
- net SPI_SCK: now also J8.7 (P7)
- net TFT_CS: now also J8.3 (P3)
- net TFT_DC: now also J8.5 (P5)
- net TFT_RST: now also J8.4 (P4)
- net TOUCH_CS: now also J8.10 (P10)
- net TOUCH_IRQ: now also J8.11 (P11)

Commit message: Wiecej RJ45 (8 podwojnych=64 wej), zabezpieczenia, zlacza na obu krawedziach
- Wejscia: 8 podwojnych RJ45 = 16 portow = 64 wejscia (4 ekspandery MCP23017).
- Zabezpieczenia: PTC na kazde z 16 wyjsc, MOV na wyjsciach 230V, snubber RC na
  stykach przekaznikow, dlawik wspolny (CMC) + TVS na RS485/CAN, TVS na wyjsciach DC.
  Nowe czesci: PTC (polyfuse), CMC (common-mode choke).
- Layout: zlacza rozlozone na GORNA i DOLNA krawedz (_split_balanced) -> wezsza
  plytka; gestsze upakowanie, mniejszy luz wysokosci. auto_frame liczy szerokosc
  z rozlozenia na 2 krawedzie. HomeCtrlPro: 237 -> 155 mm szerokosci.

Oba PCB 0/0/0, testy 12/12, kiutils OK.

Co-Authored-By: Claude Opus 4.8 (1M context) <noreply@anthropic.com>
Claude-Session: https://claude.ai/code/session_01LNGxtK2Jv1rJLBLPTwFQ9C
Parts:
- removed J6: RS485, pcbforge:RJ45_8P8C, symbol pcbforge:RJ45_8P8C
- removed J7: CAN, pcbforge:RJ45_8P8C, symbol pcbforge:RJ45_8P8C
- removed J8: TFT, pcbforge:Header_1x14, symbol pcbforge:Header_1x14
- removed U4: MAX485, pcbforge:SOIC-8, symbol pcbforge:MAX485
- removed U5: TJA1051, pcbforge:SOIC-8, symbol pcbforge:TJA1051
- added C10, C9: 100nF, pcbforge:C_0805, symbol pcbforge:C
- added D37, D38, D39, D40, D41, D42, D43, D44, D45, D46, D47, D48, D49, D50, D51, D52, D53, D54, D55, D56, D57, D58, D59, D60, D61, D62, D63, D64: ESD, pcbforge:D_SOD-323, symbol pcbforge:D_TVS
- added D65, D66, D67, D68: TVS, pcbforge:D_SOD-323, symbol pcbforge:D_TVS
- added J10: RS485, pcbforge:RJ45_8P8C, symbol pcbforge:RJ45_8P8C
- added J11: CAN, pcbforge:RJ45_8P8C, symbol pcbforge:RJ45_8P8C
- added J12: TFT, pcbforge:Header_1x14, symbol pcbforge:Header_1x14
- added J6: We 32-39, pcbforge:RJ45_Dual, symbol pcbforge:RJ45_Dual
- added J7: We 40-47, pcbforge:RJ45_Dual, symbol pcbforge:RJ45_Dual
- added J8: We 48-55, pcbforge:RJ45_Dual, symbol pcbforge:RJ45_Dual
- added J9: We 56-63, pcbforge:RJ45_Dual, symbol pcbforge:RJ45_Dual
- added L1, L2: CMC, pcbforge:CMC_4, symbol pcbforge:CMC
- added U4, U5: MCP23017, pcbforge:SOIC-28, symbol pcbforge:MCP23017
- added U6: MAX485, pcbforge:SOIC-8, symbol pcbforge:MAX485
- added U7: TJA1051, pcbforge:SOIC-8, symbol pcbforge:TJA1051
- D33, D34, D35, D36: value TVS -> ESD
Connections:
- net 3V3: now also C10.1, C9.1, J10.7 (P7), J10.8 (P8), J11.7 (P7), J11.8 (P8), J12.14 (P14), J12.2 (P2), J12.8 (P8), J6.1 (A1), J6.9 (B1), J7.1 (A1), J7.9 (B1), J8.1 (A1), J8.9 (B1), J9.1 (A1), J9.9 (B1), U4.16 (A1), U4.9 (VDD), U5.15 (A0), U5.16 (A1), U5.9 (VDD), U6.8 (VCC), U7.3 (VCC), U7.5 (VIO)
- net CAN_H: now also L2.1 (A1), U7.7 (CANH); no longer D35.1
- net CAN_L: now also L2.4 (B1), U7.6 (CANL); no longer D36.1
- net CAN_RXD: now also U7.4 (RXD)
- net CAN_TXD: now also U7.1 (TXD)
- net EXP_INT: now also U4.20 (INTA), U5.20 (INTA)
- net EXP_RST: now also U4.18 (RESET), U5.18 (RESET)
- net GND: now also C10.2, C9.2, D37.2, D38.2, D39.2, D40.2, D41.2, D42.2, D43.2, D44.2, D45.2, D46.2, D47.2, D48.2, D49.2, D50.2, D51.2, D52.2, D53.2, D54.2, D55.2, D56.2, D57.2, D58.2, D59.2, D60.2, D61.2, D62.2, D63.2, D64.2, D65.2, D66.2, D67.2, D68.2, J10.3 (P3), J10.4 (P4), J10.5 (P5), J10.6 (P6), J10.S (SHIELD), J11.3 (P3), J11.4 (P4), J11.5 (P5), J11.6 (P6), J11.S (SHIELD), J12.1 (P1), J12.13 (P13), J6.14 (B6), J6.15 (B7), J6.16 (B8), J6.6 (A6), J6.7 (A7), J6.8 (A8), J6.S (SHIELD), J7.14 (B6), J7.15 (B7), J7.16 (B8), J7.6 (A6), J7.7 (A7), J7.8 (A8), J7.S (SHIELD), J8.14 (B6), J8.15 (B7), J8.16 (B8), J8.6 (A6), J8.7 (A7), J8.8 (A8), J8.S (SHIELD), J9.14 (B6), J9.15 (B7), J9.16 (B8), J9.6 (A6), J9.7 (A7), J9.8 (A8), J9.S (SHIELD), U4.10 (VSS), U4.15 (A0), U4.17 (A2), U5.10 (VSS), U5.17 (A2), U6.5 (GND), U7.2 (GND), U7.8 (STB)
- net RS485_A: now also L1.1 (A1), U6.6 (A); no longer D33.1
- net RS485_B: now also L1.4 (B1), U6.7 (B); no longer D34.1
- net RS485_DE: now also U6.2 (RE), U6.3 (DE)
- net RS485_RXD: now also U6.1 (RO)
- net RS485_TXD: now also U6.4 (DI)
- net SCL: now also U4.12 (SCL), U5.12 (SCL)
- net SDA: now also U4.13 (SDA), U5.13 (SDA)
- net SPI_MISO: now also J12.12 (P12), J12.9 (P9)
- net SPI_MOSI: now also J12.6 (P6)
- net SPI_SCK: now also J12.7 (P7)
- net TFT_CS: now also J12.3 (P3)
- net TFT_DC: now also J12.5 (P5)
- net TFT_RST: now also J12.4 (P4)
- net TOUCH_CS: now also J12.10 (P10)
- net TOUCH_IRQ: now also J12.11 (P11)
- new net CAN_H_O: D67.1, J11.1 (P1), L2.2 (A2)
- new net CAN_L_O: D68.1, J11.2 (P2), L2.3 (B2)
- new net IN32: D33.1, J6.2 (A2), U4.21 (GPA0)
- new net IN33: D34.1, J6.3 (A3), U4.22 (GPA1)
- new net IN34: D35.1, J6.4 (A4), U4.23 (GPA2)
- new net IN35: D36.1, J6.5 (A5), U4.24 (GPA3)
- new net IN36: D37.1, J6.10 (B2), U4.25 (GPA4)
- new net IN37: D38.1, J6.11 (B3), U4.26 (GPA5)
- new net IN38: D39.1, J6.12 (B4), U4.27 (GPA6)
- new net IN39: D40.1, J6.13 (B5), U4.28 (GPA7)
- new net IN40: D41.1, J7.2 (A2), U4.1 (GPB0)
- new net IN41: D42.1, J7.3 (A3), U4.2 (GPB1)
- new net IN42: D43.1, J7.4 (A4), U4.3 (GPB2)
- new net IN43: D44.1, J7.5 (A5), U4.4 (GPB3)
- new net IN44: D45.1, J7.10 (B2), U4.5 (GPB4)
- new net IN45: D46.1, J7.11 (B3), U4.6 (GPB5)
- new net IN46: D47.1, J7.12 (B4), U4.7 (GPB6)
- new net IN47: D48.1, J7.13 (B5), U4.8 (GPB7)
- new net IN48: D49.1, J8.2 (A2), U5.21 (GPA0)
- new net IN49: D50.1, J8.3 (A3), U5.22 (GPA1)
- new net IN50: D51.1, J8.4 (A4), U5.23 (GPA2)
- new net IN51: D52.1, J8.5 (A5), U5.24 (GPA3)
- new net IN52: D53.1, J8.10 (B2), U5.25 (GPA4)
- new net IN53: D54.1, J8.11 (B3), U5.26 (GPA5)
- new net IN54: D55.1, J8.12 (B4), U5.27 (GPA6)
- new net IN55: D56.1, J8.13 (B5), U5.28 (GPA7)
- new net IN56: D57.1, J9.2 (A2), U5.1 (GPB0)
- new net IN57: D58.1, J9.3 (A3), U5.2 (GPB1)
- new net IN58: D59.1, J9.4 (A4), U5.3 (GPB2)
- new net IN59: D60.1, J9.5 (A5), U5.4 (GPB3)
- new net IN60: D61.1, J9.10 (B2), U5.5 (GPB4)
- new net IN61: D62.1, J9.11 (B3), U5.6 (GPB5)
- new net IN62: D63.1, J9.12 (B4), U5.7 (GPB6)
- new net IN63: D64.1, J9.13 (B5), U5.8 (GPB7)
- new net RS485_A_O: D65.1, J10.1 (P1), L1.2 (A2)
- new net RS485_B_O: D66.1, J10.2 (P2), L1.3 (B2)

Commit message: Zageszczenie layoutu: ~2x mniejsza plytka (zajetosc 18% -> 38%)
- Pakowanie sortowane po wysokosci (wiersze o zblizonej wysokosci) - koniec z
  marnowaniem miejsca przez wysoki element w rzedzie.
- io_band = male wciecie (nie wysokosc zlacza); wysokie podwojne RJ45 mieszcza
  sie w srodku, nie rozdmuchuja pasow krawedziowych.
- Niezalezne wysokosci plyt (auto_layout) przy WSPOLNYCH otworach i B2B - mniejsza
  plyta nie dziedziczy wysokosci wiekszej.
- Wnetrze + przekazniki jako jeden ciasny blok; szerokosc wnetrza w estymacie =
  rzeczywista (koniec z przeszacowana wysokoscia/luka).
- Wysokie zlacza grupowane na jedna krawedz; TFT 2x07 (polowa szerokosci).

HomeCtrlPro DOL: 280x185 -> 168x100 mm. Oba 0/0/0, testy 12/12, kiutils OK.

Co-Authored-By: Claude Opus 4.8 (1M context) <noreply@anthropic.com>
Claude-Session: https://claude.ai/code/session_01LNGxtK2Jv1rJLBLPTwFQ9C
Parts:
- removed J12: TFT, pcbforge:Header_1x14, symbol pcbforge:Header_1x14
- added J12: TFT, pcbforge:Header_2x07, symbol pcbforge:Header_2x07
Connections:
- net 3V3: now also J12.14 (P14), J12.2 (P2), J12.8 (P8)
- net GND: now also J12.1 (P1), J12.13 (P13)
- net SPI_MISO: now also J12.12 (P12), J12.9 (P9)
- net SPI_MOSI: now also J12.6 (P6)
- net SPI_SCK: now also J12.7 (P7)
- net TFT_CS: now also J12.3 (P3)
- net TFT_DC: now also J12.5 (P5)
- net TFT_RST: now also J12.4 (P4)
- net TOUCH_CS: now also J12.10 (P10)
- net TOUCH_IRQ: now also J12.11 (P11)
